Commit message: 🛠️ Redesign AGV URDF

File: description/gazebo_control.xacro (robot description, xacro)
@@ -6,9 +6,9 @@
             <left_joint>left_wheel_joint</left_joint>
             <right_joint>right_wheel_joint</right_joint>
-            <wheel_separation>0.393</wheel_separation>
-            <wheel_diameter>0.066</wheel_diameter>
+            <wheel_separation>0.828</wheel_separation>
+            <wheel_diameter>0.172</wheel_diameter>
             <!-- Limits -->
-            <max_wheel_torque>400</max_wheel_torque> <!-- 200 -->
-            <max_wheel_acceleration>50</max_wheel_acceleration> <!-- 10 -->
+            <max_wheel_torque>200</max_wheel_torque> <!-- 200 -->
+            <max_wheel_acceleration>10</max_wheel_acceleration> <!-- 10 -->
             <!-- Output -->
             <odometry_frame>odom</odometry_frame>

File: description/robot_core.xacro (robot description, xacro)
@@ -17,78 +17,78 @@
     </joint>
     <link name="chassi">
+    <inertial>
+        <origin xyz="0.27608648550801496 0.20950044976760585 0.1266980632048793" rpy="0 0 0"/>
+        <mass value="185.8858323610559"/>
+        <inertia ixx="2.96664" iyy="4.920526" izz="7.391448" ixy="-1.1e-05" iyz="-3.5e-05" ixz="-0.268903"/>
+    </inertial>
+    <visual>
+        <origin xyz="0 0 0" rpy="0 0 0"/>
+        <geometry>
+            <mesh filename="file://$(find agv_lince)/meshes/chassi.stl" scale="0.001 0.001 0.001"/>
+        </geometry>
+        <material name="silver"/>
+    </visual>
+    <collision>
+        <origin xyz="0 0 0" rpy="0 0 0"/>
+        <geometry>
+            <mesh filename="file://$(find agv_lince)/meshes/chassi.stl" scale="0.001 0.001 0.001"/>
+        </geometry>
+    </collision>
+    </link>
+    <!-- Left Caster -->
+    <joint name="left_caster_joint" type="fixed">
+        <origin xyz="0.5255 0.336269 0.1322" rpy="0 0 0"/>
+        <parent link="chassi"/>
+        <child link="left_caster"/>
+    </joint>
+    <link name="left_caster">
         <inertial>
-            <origin rpy="0 0 0" xyz="0.005723690556912747 -1.2710837581631485e-16 0.1330365108864905"/>
-            <mass value="49.457223713872615"/>
-            <inertia ixx="0.894743" ixy="0.0" ixz="-0.06522" iyy="2.245921" iyz="-0.0" izz="2.9822"/>
+            <origin xyz="0.0002703596792763552 2.5251487542454765e-05 -0.06165617323973693" rpy="0 0 0"/>
+            <mass value="5.442426439867197"/>
+            <inertia ixx="0.013498" iyy="0.015226" izz="0.00705" ixy="-1e-06" iyz="1e-05" ixz="6.6e-05"/>
         </inertial>
         <visual>
-            <origin rpy="0 0 0" xyz="0 0 0"/>
+            <origin xyz="-0.5255 -0.336269 -0.1322" rpy="0 0 0"/>
             <geometry>
-                <mesh filename="file://$(find agv_lince)/meshes/base_link.stl" scale="0.001 0.001 0.001"/>
+                <mesh filename="file://$(find agv_lince)/meshes/left_caster_1.stl" scale="0.001 0.001 0.001"/>
             </geometry>
             <material name="silver"/>
         </visual>
         <collision>
-            <origin rpy="0 0 0" xyz="0 0 0"/>
+            <origin xyz="-0.5255 -0.336269 -0.1322" rpy="0 0 0"/>
             <geometry>
-                <mesh filename="file://$(find agv_lince)/meshes/base_link.stl" scale="0.001 0.001 0.001"/>
+                <mesh filename="file://$(find agv_lince)/meshes/left_caster_1.stl" scale="0.001 0.001 0.001"/>
             </geometry>
         </collision>
     </link>
-    <!-- LIDAR LINK -->
-    <joint name="lidar_joint" type="fixed">
-        <origin rpy="0 0 0" xyz="0.3525 0.0 0.2655"/>
+    <!-- Right Caster -->
+    <joint name="right_caster_joint" type="fixed">
+        <origin xyz="0.5255 0.075954 0.1322" rpy="0 0 0"/>
         <parent link="chassi"/>
-        <child link="lidar"/>
+        <child link="right_caster"/>
     </joint>
-    <link name="lidar">
+    <link name="right_caster">
         <inertial>
-            <origin rpy="0 0 0" xyz="-0.000712584576985309 -4.130231120300454e-06 0.01895652806211956"/>
-            <mass value="0.17371795569954332"/>
-            <inertia ixx="8.1e-05" ixy="0.0" ixz="1e-06" iyy="7.9e-05" iyz="0.0" izz="0.000114"/>
+            <origin xyz="0.00027035967927580007 0.00033953726364627235 -0.06165617323973689" rpy="0 0 0"/>
+                <mass value="5.442426439867197"/>
+            <inertia ixx="0.013498" iyy="0.015226" izz="0.00705" ixy="-1e-06" iyz="1e-05" ixz="6.6e-05"/>
         </inertial>
         <visual>
-            <origin rpy="0 0 0" xyz="-0.3525 -0.0 -0.2655"/>
+            <origin xyz="-0.5255 -0.075954 -0.1322" rpy="0 0 0"/>
             <geometry>
-                <mesh filename="file://$(find agv_lince)/meshes/lidar_1.stl" scale="0.001 0.001 0.001"/>
+                <mesh filename="file://$(find agv_lince)/meshes/right_caster_3.stl" scale="0.001 0.001 0.001"/>
             </geometry>
             <material name="silver"/>
         </visual>
         <collision>
-            <origin rpy="0 0 0" xyz="-0.3525 -0.0 -0.2655"/>
+            <origin xyz="-0.5255 -0.075954 -0.1322" rpy="0 0 0"/>
             <geometry>
-                <mesh filename="file://$(find agv_lince)/meshes/lidar_1.stl" scale="0.001 0.001 0.001"/>
+                <mesh filename="file://$(find agv_lince)/meshes/right_caster_3.stl" scale="0.001 0.001 0.001"/>
             </geometry>
         </collision>
     </link>
-    <!-- KINECT CAMERA LINK -->
-    <joint name="kinect_joint" type="fixed">
-        <origin rpy="0 0 0" xyz="0.3555 0.0 0.1795"/>
-        <parent link="chassi"/>
-        <child link="kinect"/>
-    </joint>
-    <link name="kinect">
-        <inertial>
-            <origin rpy="0 0 0" xyz="-0.002248529840528868 4.525712411141205e-05 0.04507302819784481"/>
-            <mass value="0.6981884785115198"/>
-            <inertia ixx="0.003322" ixy="-1e-06" ixz="4e-06" iyy="0.000442" iyz="-0.0" izz="0.003298"/>
-        </inertial>
-        <visual>
-            <origin rpy="0 0 0" xyz="-0.3555 -0.0 -0.1795"/>
-            <geometry>
-                <mesh filename="file://$(find agv_lince)/meshes/kinect_1.stl" scale="0.001 0.001 0.001"/>
-            </geometry>
-            <material name="silver"/>
-        </visual>
-        <collision>
-            <origin rpy="0 0 0" xyz="-0.3555 -0.0 -0.1795"/>
-            <geometry>
-                <mesh filename="file://$(find agv_lince)/meshes/kinect_1.stl" scale="0.001 0.001 0.001"/>
-            </geometry>
-        </collision>
-    </link>
-        <!-- LEFT WHEEL LINK -->
+    <!-- Left Wheel -->
     <joint name="left_wheel_joint" type="continuous">
-        <origin rpy="0 0 0" xyz="-0.23 0.1965 0.084"/>
+        <origin xyz="0.086098 0.414 0.0522" rpy="0 0 0"/>
         <parent link="chassi"/>
         <child link="left_wheel"/>
@@ -97,10 +97,10 @@
     <link name="left_wheel">
     <inertial>
-        <origin rpy="0 0 0" xyz="2.4702462297909733e-15 0.039917522857950805 0.0"/>
-        <mass value="1.2398446203839488"/>
-        <inertia ixx="0.002557" ixy="0.0" ixz="0.0" iyy="0.004364" iyz="0.0" izz="0.002557"/>
+        <origin xyz="-2.7028745609725124e-07 0.03596400994364629 -6.938893903907228e-18" rpy="0 0 0"/>
+        <mass value="11.320743431486168"/>
+        <inertia ixx="0.024546" iyy="0.04182" izz="0.024546" ixy="-0.0" iyz="-0.0" ixz="0.0"/>
     </inertial>
     <visual>
-        <origin rpy="0 0 0" xyz="0.23 -0.1965 -0.084"/>
+        <origin xyz="-0.086098 -0.414 -0.0522" rpy="0 0 0"/>
         <geometry>
             <mesh filename="file://$(find agv_lince)/meshes/left_wheel_1.stl" scale="0.001 0.001 0.001"/>
@@ -109,5 +109,5 @@
     </visual>
     <collision>
-        <origin rpy="0 0 0" xyz="0.23 -0.1965 -0.084"/>
+        <origin xyz="-0.086098 -0.414 -0.0522" rpy="0 0 0"/>
         <geometry>
             <mesh filename="file://$(find agv_lince)/meshes/left_wheel_1.stl" scale="0.001 0.001 0.001"/>
@@ -115,30 +115,30 @@
     </collision>
     </link>
-    <!-- RIGHT WHEEL LINK -->
+    <!-- Right Wheel -->
     <joint name="right_wheel_joint" type="continuous">
-        <origin rpy="0 0 0" xyz="-0.23 -0.1965 0.084"/>
+        <origin xyz="0.082222 0.005 0.066" rpy="0 0 0"/>
         <parent link="chassi"/>
         <child link="right_wheel"/>
-        <axis xyz="-0.0 1.0 0.0"/>
+        <axis xyz="0.0 1.0 0.0"/>
     </joint>
     <link name="right_wheel">
-        <inertial>
-            <origin rpy="0 0 0" xyz="1.482147737874584e-14 -0.03991752285795086 1.3877787807814457e-17"/>
-            <mass value="1.2398446203839475"/>
-            <inertia ixx="0.002557" ixy="-0.0" ixz="0.0" iyy="0.004364" iyz="-0.0" izz="0.002557"/>
-        </inertial>
-        <visual>
-            <origin rpy="0 0 0" xyz="0.23 0.1965 -0.084"/>
-            <geometry>
-                <mesh filename="file://$(find agv_lince)/meshes/right_wheel_1.stl" scale="0.001 0.001 0.001"/>
-            </geometry>
-            <material name="silver"/>
-        </visual>
-        <collision>
-            <origin rpy="0 0 0" xyz="0.23 0.1965 -0.084"/>
-            <geometry>
-                <mesh filename="file://$(find agv_lince)/meshes/right_wheel_1.stl" scale="0.001 0.001 0.001"/>
-            </geometry>
-        </collision>
+    <inertial>
+        <origin xyz="-1.1151555552590953e-07 -0.03596400940058405 0.0" rpy="0 0 0"/>
+        <mass value="11.32074361520196"/>
+        <inertia ixx="0.024546" iyy="0.04182" izz="0.024546" ixy="-0.0" iyz="-0.0" ixz="0.0"/>
+    </inertial>
+    <visual>
+        <origin xyz="-0.082222 -0.005 -0.066" rpy="0 0 0"/>
+        <geometry>
+            <mesh filename="file://$(find agv_lince)/meshes/right_wheel_1.stl" scale="0.001 0.001 0.001"/>
+        </geometry>
+        <material name="silver"/>
+    </visual>
+    <collision>
+        <origin xyz="-0.082222 -0.005 -0.066" rpy="0 0 0"/>
+        <geometry>
+            <mesh filename="file://$(find agv_lince)/meshes/right_wheel_1.stl" scale="0.001 0.001 0.001"/>
+        </geometry>
+    </collision>
     </link>
 </robot>
