Commit message: 🔧 Add Camera to URDF

File: description/robot_core.xacro (robot description, xacro)
@@ -17,22 +17,22 @@
     </joint>
     <link name="chassi">
-    <inertial>
-        <origin xyz="0.27608648550801496 0.20950044976760585 0.1266980632048793" rpy="0 0 0"/>
-        <mass value="185.8858323610559"/>
-        <inertia ixx="2.96664" iyy="4.920526" izz="7.391448" ixy="-1.1e-05" iyz="-3.5e-05" ixz="-0.268903"/>
-    </inertial>
-    <visual>
-        <origin xyz="0 0 0" rpy="0 0 0"/>
-        <geometry>
-            <mesh filename="file://$(find agv_lince)/meshes/chassi.stl" scale="0.001 0.001 0.001"/>
-        </geometry>
-        <material name="silver"/>
-    </visual>
-    <collision>
-        <origin xyz="0 0 0" rpy="0 0 0"/>
-        <geometry>
-            <mesh filename="file://$(find agv_lince)/meshes/chassi.stl" scale="0.001 0.001 0.001"/>
-        </geometry>
-    </collision>
+        <inertial>
+            <origin xyz="0.26852392239431533 0.20950930054137695 0.1415018788660424" rpy="0 0 0"/>
+            <mass value="196.71182920620697"/>
+            <inertia ixx="4.100554" iyy="6.971657" izz="8.324299" ixy="0.000441" iyz="-0.000438" ixz="0.423937"/>
+        </inertial>
+        <visual>
+            <origin xyz="0 0 0" rpy="0 0 0"/>
+            <geometry>
+                <mesh filename="file://$(find agv_lince)/meshes/chassi.stl" scale="0.001 0.001 0.001"/>
+            </geometry>
+            <material name="silver"/>
+        </visual>
+        <collision>
+            <origin xyz="0 0 0" rpy="0 0 0"/>
+            <geometry>
+                <mesh filename="file://$(find agv_lince)/meshes/chassi.stl" scale="0.001 0.001 0.001"/>
+            </geometry>
+        </collision>
     </link>
     <!-- Left Caster -->
@@ -142,3 +142,29 @@
     </collision>
     </link>
+    <!-- Camera -->
+    <joint name="R gido 12" type="fixed">
+        <origin xyz="0.65505 0.2095 0.2277" rpy="0 0 0"/>
+        <parent link="chassi"/>
+        <child link="camera_1"/>
+    </joint>
+    <link name="camera_1">
+        <inertial>
+            <origin xyz="-0.006290550800018169 -3.1499090842684874e-05 0.036766020010442935" rpy="0 0 0"/>
+            <mass value="3.5762687778267663"/>
+            <inertia ixx="0.003848" iyy="0.003414" izz="0.004063" ixy="6e-06" iyz="1e-06" ixz="6.9e-05"/>
+        </inertial>
+        <visual>
+            <origin xyz="-0.65505 -0.2095 -0.2277" rpy="0 0 0"/>
+            <geometry>
+                <mesh filename="file://$(find agv_lince)/meshes/camera_1.stl" scale="0.001 0.001 0.001"/>
+            </geometry>
+            <material name="silver"/>
+        </visual>
+        <collision>
+            <origin xyz="-0.65505 -0.2095 -0.2277" rpy="0 0 0"/>
+            <geometry>
+                <mesh filename="file:/;$(find agv_lince)/meshes/camera_1.stl" scale="0.001 0.001 0.001"/>
+            </geometry>
+        </collision>
+    </link>
 </robot>
