Commit message: ✨ Add gazebo diff_drive control

File: description/robot.urdf.xacro (robot description, xacro)
@@ -3,3 +3,4 @@
     <xacro:include filename="robot_core.xacro" />
     <xacro:include filename="$(find agv_lince)/description/robot.gazebo" />
+    <xacro:include filename="gazebo_control.xacro" />
 </robot>

File: description/robot_core.xacro (robot description, xacro)
@@ -104,5 +104,5 @@
         <origin rpy="0 0 0" xyz="0.23 -0.1965 -0.084"/>
         <geometry>
-        <mesh filename="file://$(find agv_lince)/meshes/left_wheel_1.stl" scale="0.001 0.001 0.001"/>
+            <mesh filename="file://$(find agv_lince)/meshes/left_wheel_1.stl" scale="0.001 0.001 0.001"/>
         </geometry>
         <material name="silver"/>
@@ -111,5 +111,5 @@
         <origin rpy="0 0 0" xyz="0.23 -0.1965 -0.084"/>
         <geometry>
-        <mesh filename="file://$(find agv_lince)/meshes/left_wheel_1.stl" scale="0.001 0.001 0.001"/>
+            <mesh filename="file://$(find agv_lince)/meshes/left_wheel_1.stl" scale="0.001 0.001 0.001"/>
         </geometry>
     </collision>

Commit message: ✨ Add lidar to Gazebo Sim

File: description/robot.urdf.xacro (robot description, xacro)
@@ -5,3 +5,4 @@
     <!-- <xacro:include filename="gazebo_control.xacro" /> -->
     <xacro:include filename="ros2_control.xacro" />
+    <xacro:include filename="lidar.xacro" />
 </robot>

File: description/robot_core.xacro (robot description, xacro)
@@ -143,5 +143,5 @@
     </link>
     <!-- Camera -->
-    <joint name="R gido 12" type="fixed">
+    <!-- <joint name="R gido 12" type="fixed">
         <origin xyz="0.65505 0.2095 0.2277" rpy="0 0 0"/>
         <parent link="chassi"/>
@@ -167,4 +167,4 @@
             </geometry>
         </collision>
-    </link>
+    </link> -->
 </robot>
